Commit message: Fixed camera mesh and consolidated to a single file.

File: robots/hubo_head_description.URDF (robot description, URDF)
Before this commit: robot hubo_head_description, 9 links, 8 joints
Links:
- link camera_c_link: geometry collision mesh filename=package://hubo_head_description/meshes/flea_camera.STL; visual mesh filename=package://hubo_head_description/meshes/flea_camera.STL
- link camera_l_link: geometry collision mesh filename=package://hubo_head_description/meshes/flea_camera.STL; visual mesh filename=package://hubo_head_description/meshes/flea_camera.STL
- link camera_r_link: geometry collision mesh filename=package://hubo_head_description/meshes/flea_camera.STL; visual mesh filename=package://hubo_head_description/meshes/flea_camera.STL

Commit message: Added optical frame for Hokuyo.

File: robots/hubo_head_description.URDF (robot description, URDF)
Before this commit: robot hubo_head_description, 9 links, 8 joints
Links:
- added link lidar_optical_frame
Joints:
- added joint lidar_optical_link: type fixed, parent lidar_tilt_link, child lidar_optical_frame, origin xyz=0 0.0375 0.00135 rpy=1.5708 -1.0106E-15 3.1416, axis 0 0 0

Commit message: Updated joint axes to be consistent with convention at home position.

File: robots/hubo_head_description.URDF (robot description, URDF)
Before this commit: robot hubo_head_description, 10 links, 9 joints
Links:
- link camera_c_link: mass 0.059131 -> 0.0591308427749407
- link camera_l_link: mass 0.059131 -> 0.059130842653584
- link camera_r_link: mass 0.059131 -> 0.0591308428004722
- link head_base_link: mass 0.022215 -> 0.0222146018366026
- link lidar_tilt_link: mass 0.27744 -> 0.277440816169479
- link turret_pan_link: mass 0.11166 -> 0.111664559813447
- link turret_tilt_link: mass 0.95331 -> 0.953306948960365
Joints:
- joint camera_c: origin xyz=0.040455 0.028675 0.14586 rpy=0 0 0 -> xyz=0.040455 0.028675 0.14036 rpy=0 0 0
- joint camera_l: origin xyz=0.040455 0.088675 0.14586 rpy=0 0 0 -> xyz=0.040455 0.088675 0.14036 rpy=0 0 0
- joint camera_r: origin xyz=0.040455 -0.091325 0.14586 rpy=0 0 0 -> xyz=0.040455 -0.091325 0.14036 rpy=0 0 0
- joint lidar_optical_link: origin xyz=0 0.0375 0.00135 rpy=1.5708 -1.0106E-15 3.1416 -> xyz=0 0.00134999999999998 0.032 rpy=0 0 0
- joint lidar_tilt: axis 0 0 -1 -> 0 -1 0; origin xyz=0.062 0 0.03636 rpy=1.5707963267949 1.62525199293825E-31 3.14159265358979 -> xyz=0.062 0 0.03636 rpy=0 0 0
- joint ps_lower_base: origin xyz=-0.067789086884583 -0.00132499999999999 0.125855390601482 rpy=8.13589349446095E-16 0.747175452778788 -3.14159265358979 -> xyz=-0.067789086884583 -0.00132499999999999 0.120355390601482 rpy=8.13589349446095E-16 0.747175452778788 -3.14159265358979
- joint ps_upper_base: origin xyz=-0.068045 -0.00132499999999995 0.175676213379847 rpy=5.96858314644388E-16 1.04083408558608E-15 3.14159265358979 -> xyz=-0.068045 -0.00132499999999995 0.170176213379847 rpy=5.96858314644388E-16 1.04083408558608E-15 3.14159265358979
- joint turret_pan: axis 0 0 -1 -> 0 0 1; origin xyz=0 0 0 rpy=3.14159265358979 0 1.5707963267949 -> xyz=0 0 0 rpy=0 0 0
- joint turret_tilt: origin xyz=0 0 -0.0755 rpy=-3.14159265358979 -1.21972744404619E-16 1.5707963267949 -> xyz=0 0 0.081 rpy=0 0 0

Commit message: Corrected lidar axis direction and neck offset.

File: robots/hubo_head_description.URDF (robot description, URDF)
Before this commit: robot hubo_head_description, 10 links, 9 joints
Joints:
- joint lidar_tilt: axis 0 -1 0 -> 0 1 0

Commit message: Changes made on vision laptop

File: robots/hubo_head_description.URDF (robot description, URDF)
Before this commit: robot hubo_head_description, 10 links, 9 joints
Links:
- removed link ps_lower_base_link
- removed link ps_upper_base_link
- added link camera_c_optical_frame
- added link camera_l_optical_frame
- added link camera_r_optical_frame
- link camera_c_link: mass 0.0591308427749407 -> 0.0591308424717379
- link camera_l_link: mass 0.059130842653584 -> 0.0591308426614994
- link camera_r_link: mass 0.0591308428004722 -> 0.0591308423327651
- link turret_pan_link: mass 0.111664559813447 -> 0.109664559813447
- link turret_tilt_link: mass 0.953306948960365 -> 0.570110653946282
Joints:
- removed joint ps_lower_base
- removed joint ps_upper_base
- added joint camera_c_optical: type fixed, parent camera_c_link, child camera_c_optical_frame, origin xyz=0 0 0 rpy=-1.5707963267949 -1.17497412307793E-15 -1.5707963267949, axis 0 0 0
- added joint camera_l_optical: type fixed, parent camera_l_link, child camera_l_optical_frame, origin xyz=0 0 0 rpy=-1.5707963267949 -9.89729612979842E-16 -1.5707963267949, axis 0 0 0
- added joint camera_r_optical: type fixed, parent camera_r_link, child camera_r_optical_frame, origin xyz=0 0 0 rpy=-1.5707963267949 -3.50979685635337E-16 -1.5707963267949, axis 0 0 0
- joint camera_c: origin xyz=0.040455 0.028675 0.14036 rpy=0 0 0 -> xyz= 0.05319  0.02597  0.13636 rpy= 0.01860 -0.00031  0.00006
- joint camera_l: origin xyz=0.040455 0.088675 0.14036 rpy=0 0 0 -> xyz=0.015955 0.0923500000000001 0.14036 rpy=0 0 0
- joint camera_r: origin xyz=0.040455 -0.091325 0.14036 rpy=0 0 0 -> xyz=-0.03 -0.08765 0.14036 rpy=0.018 -0.01 0.03
- joint lidar_optical_link: origin xyz=0 0.00134999999999998 0.032 rpy=0 0 0 -> xyz=0 -0.00108907916431705 0.0320031382660522 rpy=-0.00276893204593277 1.38777346074552E-15 -3.84266022849734E-18
- joint lidar_tilt: axis 0 1 0 -> 0 1 0.00276892850770753; origin xyz=0.062 0 0.03636 rpy=0 0 0 -> xyz=0.062 2.76893912240783E-05 0.03636 rpy=0.00276893204593277 -1.38777878078144E-15 0
